File: Futai Encoder + WS2811 ring.kicad_sch (KiCad schematic)
At the start: 41 parts, among them J1 Conn_02x05_Top_Bottom, SW1 RotaryEncoder_Switch_RGB

Commit message: smaller board width, new component placements and better track routing
Parts:
- R1, R10, R11, R12, R2, R3, R4, R5, R6, R7, R8, R9: value 160 -> 130
Changed lines of the file:
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@@
   (title_block
     (title "enlighted rotary encoder")
-    (date "2022-01-01")
-    (rev "0.5")
+    (date "2022-01-04")
+    (rev "0.65")
     (company "designed by andilge")
   )
@@
     (in_bom yes) (on_board yes) (fields_autoplaced)
     (property "Reference" "R8" (id 0) (at 102.87 95.25 90))
-    (property "Value" "160" (id 1) (at 102.87 97.79 90))
+    (property "Value" "130" (id 1) (at 102.87 97.79 90))
     (property "Footprint" "Resistor_SMD:R_0805_2012Metric" (id 2) (at 102.87 101.6 0)
       (effects (font (size 1.27 1.27)) hide)
@@
     (in_bom yes) (on_board yes) (fields_autoplaced)
     (property "Reference" "R10" (id 0) (at 120.65 125.73 90))
-    (property "Value" "160" (id 1) (at 120.65 128.27 90))
+    (property "Value" "130" (id 1) (at 120.65 128.27 90))
     (property "Footprint" "Resistor_SMD:R_0805_2012Metric" (id 2) (at 120.65 132.08 0)
       (effects (font (size 1.27 1.27)) hide)
@@
     (in_bom yes) (on_board yes) (fields_autoplaced)
     (property "Reference" "R3" (id 0) (at 120.65 34.29 90))
-    (property "Value" "160" (id 1) (at 120.65 36.83 90))
+    (property "Value" "130" (id 1) (at 120.65 36.83 90))
     (property "Footprint" "Resistor_SMD:R_0805_2012Metric" (id 2) (at 120.65 40.64 0)
       (effects (font (size 1.27 1.27)) hide)
@@
     (in_bom yes) (on_board yes) (fields_autoplaced)
     (property "Reference" "R5" (id 0) (at 102.87 64.77 90))
-    (property "Value" "160" (id 1) (at 102.87 67.31 90))
+    (property "Value" "130" (id 1) (at 102.87 67.31 90))
     (property "Footprint" "Resistor_SMD:R_0805_2012Metric" (id 2) (at 102.87 71.12 0)
       (effects (font (size 1.27 1.27)) hide)
@@
     (in_bom yes) (on_board yes) (fields_autoplaced)
     (property "Reference" "R6" (id 0) (at 85.09 64.77 90))
-    (property "Value" "160" (id 1) (at 85.09 67.31 90))
+    (property "Value" "130" (id 1) (at 85.09 67.31 90))
     (property "Footprint" "Resistor_SMD:R_0805_2012Metric" (id 2) (at 85.09 71.12 0)
       (effects (font (size 1.27 1.27)) hide)
@@
     (in_bom yes) (on_board yes) (fields_autoplaced)
     (property "Reference" "R9" (id 0) (at 120.65 95.25 90))
-    (property "Value" "160" (id 1) (at 120.65 97.79 90))
+    (property "Value" "130" (id 1) (at 120.65 97.79 90))
     (property "Footprint" "Resistor_SMD:R_0805_2012Metric" (id 2) (at 120.65 101.6 0)
       (effects (font (size 1.27 1.27)) hide)
@@
     (in_bom yes) (on_board yes) (fields_autoplaced)
     (property "Reference" "R1" (id 0) (at 85.09 34.29 90))
-    (property "Value" "160" (id 1) (at 85.09 36.83 90))
+    (property "Value" "130" (id 1) (at 85.09 36.83 90))
     (property "Footprint" "Resistor_SMD:R_0805_2012Metric" (id 2) (at 85.09 40.64 0)
       (effects (font (size 1.27 1.27)) hide)
@@
     (in_bom yes) (on_board yes) (fields_autoplaced)
     (property "Reference" "R4" (id 0) (at 120.65 64.77 90))
-    (property "Value" "160" (id 1) (at 120.65 67.31 90))
+    (property "Value" "130" (id 1) (at 120.65 67.31 90))
     (property "Footprint" "Resistor_SMD:R_0805_2012Metric" (id 2) (at 120.65 71.12 0)
       (effects (font (size 1.27 1.27)) hide)
@@
     (in_bom yes) (on_board yes) (fields_autoplaced)
     (property "Reference" "R12" (id 0) (at 85.09 125.73 90))
-    (property "Value" "160" (id 1) (at 85.09 128.27 90))
+    (property "Value" "130" (id 1) (at 85.09 128.27 90))
     (property "Footprint" "Resistor_SMD:R_0805_2012Metric" (id 2) (at 85.09 132.08 0)
       (effects (font (size 1.27 1.27)) hide)
@@
     (in_bom yes) (on_board yes) (fields_autoplaced)
     (property "Reference" "R2" (id 0) (at 102.87 34.29 90))
-    (property "Value" "160" (id 1) (at 102.87 36.83 90))
+    (property "Value" "130" (id 1) (at 102.87 36.83 90))
     (property "Footprint" "Resistor_SMD:R_0805_2012Metric" (id 2) (at 102.87 40.64 0)
       (effects (font (size 1.27 1.27)) hide)
@@
     (in_bom yes) (on_board yes) (fields_autoplaced)
     (property "Reference" "R11" (id 0) (at 102.87 125.73 90))
-    (property "Value" "160" (id 1) (at 102.87 128.27 90))
+    (property "Value" "130" (id 1) (at 102.87 128.27 90))
     (property "Footprint" "Resistor_SMD:R_0805_2012Metric" (id 2) (at 102.87 132.08 0)
       (effects (font (size 1.27 1.27)) hide)
@@
     (in_bom yes) (on_board yes) (fields_autoplaced)
     (property "Reference" "R7" (id 0) (at 85.09 95.25 90))
-    (property "Value" "160" (id 1) (at 85.09 97.79 90))
+    (property "Value" "130" (id 1) (at 85.09 97.79 90))
     (property "Footprint" "Resistor_SMD:R_0805_2012Metric" (id 2) (at 85.09 101.6 0)
       (effects (font (size 1.27 1.27)) hide)
@@
     )
     (path "/a1907388-9e00-468a-988b-8992902b3682"
-      (reference "R1") (unit 1) (value "160") (footprint "Resistor_SMD:R_0805_2012Metric")
+      (reference "R1") (unit 1) (value "130") (footprint "Resistor_SMD:R_0805_2012Metric")
     )
     (path "/bd29be46-488e-4e08-b4da-96638cf12682"
-      (reference "R2") (unit 1) (value "160") (footprint "Resistor_SMD:R_0805_2012Metric")
+      (reference "R2") (unit 1) (value "130") (footprint "Resistor_SMD:R_0805_2012Metric")
     )
     (path "/14453a58-5327-4949-b6fd-b66f4b436bab"
-      (reference "R3") (unit 1) (value "160") (footprint "Resistor_SMD:R_0805_2012Metric")
+      (reference "R3") (unit 1) (value "130") (footprint "Resistor_SMD:R_0805_2012Metric")
     )
     (path "/aa5c361e-15bc-43d6-86f2-1ed525ecf6c4"
-      (reference "R4") (unit 1) (value "160") (footprint "Resistor_SMD:R_0805_2012Metric")
+      (reference "R4") (unit 1) (value "130") (footprint "Resistor_SMD:R_0805_2012Metric")
     )
     (path "/777fe8f2-679b-4ab3-8661-f8ea51b30eb5"
-      (reference "R5") (unit 1) (value "160") (footprint "Resistor_SMD:R_0805_2012Metric")
+      (reference "R5") (unit 1) (value "130") (footprint "Resistor_SMD:R_0805_2012Metric")
     )
     (path "/7c6bc579-2e40-428e-8e02-8ea37e169713"
-      (reference "R6") (unit 1) (value "160") (footprint "Resistor_SMD:R_0805_2012Metric")
+      (reference "R6") (unit 1) (value "130") (footprint "Resistor_SMD:R_0805_2012Metric")
     )
     (path "/d3ee32eb-50bd-4159-b780-721a0ef3b763"
-      (reference "R7") (unit 1) (value "160") (footprint "Resistor_SMD:R_0805_2012Metric")
+      (reference "R7") (unit 1) (value "130") (footprint "Resistor_SMD:R_0805_2012Metric")
     )
     (path "/0a22ebe2-19e4-4e44-aec5-220a61f1450f"
-      (reference "R8") (unit 1) (value "160") (footprint "Resistor_SMD:R_0805_2012Metric")
+      (reference "R8") (unit 1) (value "130") (footprint "Resistor_SMD:R_0805_2012Metric")
     )
     (path "/7fdf067d-1b60-4cbc-9f7c-e330736a106f"
-      (reference "R9") (unit 1) (value "160") (footprint "Resistor_SMD:R_0805_2012Metric")
+      (reference "R9") (unit 1) (value "130") (footprint "Resistor_SMD:R_0805_2012Metric")
     )
     (path "/0f303b4e-56c5-4092-86d3-ba3d944a7183"
-      (reference "R10") (unit 1) (value "160") (footprint "Resistor_SMD:R_0805_2012Metric")
+      (reference "R10") (unit 1) (value "130") (footprint "Resistor_SMD:R_0805_2012Metric")
     )
     (path "/bdaf077b-081d-4ce2-9917-9e66a4691edd"
-      (reference "R11") (unit 1) (value "160") (footprint "Resistor_SMD:R_0805_2012Metric")
+      (reference "R11") (unit 1) (value "130") (footprint "Resistor_SMD:R_0805_2012Metric")
     )
     (path "/ab739511-7e26-470d-a2f4-e231c5b21cc6"
-      (reference "R12") (unit 1) (value "160") (footprint "Resistor_SMD:R_0805_2012Metric")
+      (reference "R12") (unit 1) (value "130") (footprint "Resistor_SMD:R_0805_2012Metric")
     )
     (path "/fa9aa5e4-b61f-4a04-b576-5b06f9fd3c52"

Commit message: completeing 3d models, adding new images
Parts:
- D1, D10, D11, D12, D2, D3, D4, D5, D6, D7, D8, D9: footprint footprints:WS2811-THT-LED -> LED_SMD:LED_WS2812D-F5-1261_5.8x8.6mm_P1.1mm
- SW1: Purchase https:/www.aliexpress.com/item/1005002478550056.html -> https://www.aliexpress.com/item/1005002478234416.html
Changed lines of the file:
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@@
       (effects (font (size 1.27 1.27)) (justify right))
     )
-    (property "Footprint" "footprints:WS2811-THT-LED" (id 2) (at 125.73 116.84 0)
+    (property "Footprint" "LED_SMD:LED_WS2812D-F5-1261_5.8x8.6mm_P1.1mm" (id 2) (at 125.73 116.84 0)
       (effects (font (size 1.27 1.27)) (justify left top) hide)
     )
@@
     (pin "2")
   )
-  (symbol (lib_name "R_Small_1") (lib_id "Device:R_Small") (at 157.48 95.25 270) (unit 1)
+  (symbol (lib_id "Device:R_Small") (at 157.48 95.25 270) (unit 1)
     (in_bom yes) (on_board yes)
     (property "Reference" "R41" (id 0) (at 157.48 90.17 90))
@@
       (effects (font (size 1.27 1.27)) (justify left))
     )
-    (property "Footprint" "footprints:WS2811-THT-LED" (id 2) (at 123.19 147.32 0)
+    (property "Footprint" "LED_SMD:LED_WS2812D-F5-1261_5.8x8.6mm_P1.1mm" (id 2) (at 123.19 147.32 0)
       (effects (font (size 1.27 1.27)) (justify left top) hide)
     )
@@
       (effects (font (size 1.27 1.27)) (justify left))
     )
-    (property "Footprint" "footprints:WS2811-THT-LED" (id 2) (at 90.17 55.88 0)
+    (property "Footprint" "LED_SMD:LED_WS2812D-F5-1261_5.8x8.6mm_P1.1mm" (id 2) (at 90.17 55.88 0)
       (effects (font (size 1.27 1.27)) (justify left top) hide)
     )
@@
       (effects (font (size 1.27 1.27)) (justify right))
     )
-    (property "Footprint" "footprints:WS2811-THT-LED" (id 2) (at 90.17 116.84 0)
+    (property "Footprint" "LED_SMD:LED_WS2812D-F5-1261_5.8x8.6mm_P1.1mm" (id 2) (at 90.17 116.84 0)
       (effects (font (size 1.27 1.27)) (justify left top) hide)
     )
@@
       (effects (font (size 1.27 1.27)) hide)
     )
-    (property "Purchase" "https:/www.aliexpress.com/item/1005002478550056.html" (id 4) (at 166.37 130.81 0)
+    (property "Purchase" "https://www.aliexpress.com/item/1005002478234416.html" (id 4) (at 166.37 130.81 0)
       (effects (font (size 1.27 1.27)) hide)
     )
@@
       (effects (font (size 1.27 1.27)) (justify left))
     )
-    (property "Footprint" "footprints:WS2811-THT-LED" (id 2) (at 107.95 55.88 0)
+    (property "Footprint" "LED_SMD:LED_WS2812D-F5-1261_5.8x8.6mm_P1.1mm" (id 2) (at 107.95 55.88 0)
       (effects (font (size 1.27 1.27)) (justify left top) hide)
     )
@@
       (effects (font (size 1.27 1.27)) (justify left))
     )
-    (property "Footprint" "footprints:WS2811-THT-LED" (id 2) (at 87.63 147.32 0)
+    (property "Footprint" "LED_SMD:LED_WS2812D-F5-1261_5.8x8.6mm_P1.1mm" (id 2) (at 87.63 147.32 0)
       (effects (font (size 1.27 1.27)) (justify left top) hide)
     )
@@
       (effects (font (size 1.27 1.27)) (justify left))
     )
-    (property "Footprint" "footprints:WS2811-THT-LED" (id 2) (at 105.41 86.36 0)
+    (property "Footprint" "LED_SMD:LED_WS2812D-F5-1261_5.8x8.6mm_P1.1mm" (id 2) (at 105.41 86.36 0)
       (effects (font (size 1.27 1.27)) (justify left top) hide)
     )
@@
       (effects (font (size 1.27 1.27)) (justify left))
     )
-    (property "Footprint" "footprints:WS2811-THT-LED" (id 2) (at 125.73 55.88 0)
+    (property "Footprint" "LED_SMD:LED_WS2812D-F5-1261_5.8x8.6mm_P1.1mm" (id 2) (at 125.73 55.88 0)
       (effects (font (size 1.27 1.27)) (justify left top) hide)
     )
@@
       (effects (font (size 1.27 1.27)) (justify left))
     )
-    (property "Footprint" "footprints:WS2811-THT-LED" (id 2) (at 105.41 147.32 0)
+    (property "Footprint" "LED_SMD:LED_WS2812D-F5-1261_5.8x8.6mm_P1.1mm" (id 2) (at 105.41 147.32 0)
       (effects (font (size 1.27 1.27)) (justify left top) hide)
     )
@@
       (effects (font (size 1.27 1.27)) (justify left))
     )
-    (property "Footprint" "footprints:WS2811-THT-LED" (id 2) (at 87.63 86.36 0)
+    (property "Footprint" "LED_SMD:LED_WS2812D-F5-1261_5.8x8.6mm_P1.1mm" (id 2) (at 87.63 86.36 0)
       (effects (font (size 1.27 1.27)) (justify left top) hide)
     )
@@
       (effects (font (size 1.27 1.27)) (justify right))
     )
-    (property "Footprint" "footprints:WS2811-THT-LED" (id 2) (at 107.95 116.84 0)
+    (property "Footprint" "LED_SMD:LED_WS2812D-F5-1261_5.8x8.6mm_P1.1mm" (id 2) (at 107.95 116.84 0)
       (effects (font (size 1.27 1.27)) (justify left top) hide)
     )
@@
       (effects (font (size 1.27 1.27)) (justify left))
     )
-    (property "Footprint" "footprints:WS2811-THT-LED" (id 2) (at 123.19 86.36 0)
+    (property "Footprint" "LED_SMD:LED_WS2812D-F5-1261_5.8x8.6mm_P1.1mm" (id 2) (at 123.19 86.36 0)
       (effects (font (size 1.27 1.27)) (justify left top) hide)
     )
@@
     )
     (path "/2d210a96-f81f-42a9-8bf4-1b43c11086f3"
-      (reference "D1") (unit 1) (value "WS2812D") (footprint "footprints:WS2811-THT-LED")
+      (reference "D1") (unit 1) (value "WS2812D") (footprint "LED_SMD:LED_WS2812D-F5-1261_5.8x8.6mm_P1.1mm")
     )
     (path "/528aa18e-2c11-4c58-a54a-78284a489bc0"
-      (reference "D2") (unit 1) (value "WS2812D") (footprint "footprints:WS2811-THT-LED")
+      (reference "D2") (unit 1) (value "WS2812D") (footprint "LED_SMD:LED_WS2812D-F5-1261_5.8x8.6mm_P1.1mm")
     )
     (path "/5f6d88dd-e418-4a2e-babb-f5b9471bb8b4"
-      (reference "D3") (unit 1) (value "WS2812D") (footprint "footprints:WS2811-THT-LED")
+      (reference "D3") (unit 1) (value "WS2812D") (footprint "LED_SMD:LED_WS2812D-F5-1261_5.8x8.6mm_P1.1mm")
     )
     (path "/f420db5b-fd00-4049-8a84-5cdee7ead735"
-      (reference "D4") (unit 1) (value "WS2812D") (footprint "footprints:WS2811-THT-LED")
+      (reference "D4") (unit 1) (value "WS2812D") (footprint "LED_SMD:LED_WS2812D-F5-1261_5.8x8.6mm_P1.1mm")
     )
     (path "/5b7bd047-6cd7-4751-978f-4daba3ab6707"
-      (reference "D5") (unit 1) (value "WS2812D") (footprint "footprints:WS2811-THT-LED")
+      (reference "D5") (unit 1) (value "WS2812D") (footprint "LED_SMD:LED_WS2812D-F5-1261_5.8x8.6mm_P1.1mm")
     )
     (path "/d9359ba8-c60c-4801-ae19-016d3a5c0bc5"
-      (reference "D6") (unit 1) (value "WS2812D") (footprint "footprints:WS2811-THT-LED")
+      (reference "D6") (unit 1) (value "WS2812D") (footprint "LED_SMD:LED_WS2812D-F5-1261_5.8x8.6mm_P1.1mm")
     )
     (path "/32c5fb38-b8ad-4351-bb6d-f583919c5bcc"
-      (reference "D7") (unit 1) (value "WS2812D") (footprint "footprints:WS2811-THT-LED")
+      (reference "D7") (unit 1) (value "WS2812D") (footprint "LED_SMD:LED_WS2812D-F5-1261_5.8x8.6mm_P1.1mm")
     )
     (path "/dbd55b71-9069-4af0-85a9-c297c32a210b"
-      (reference "D8") (unit 1) (value "WS2812D") (footprint "footprints:WS2811-THT-LED")
+      (reference "D8") (unit 1) (value "WS2812D") (footprint "LED_SMD:LED_WS2812D-F5-1261_5.8x8.6mm_P1.1mm")
     )
     (path "/05cd02a8-2260-4bbd-acde-cef32667d469"
-      (reference "D9") (unit 1) (value "WS2812D") (footprint "footprints:WS2811-THT-LED")
+      (reference "D9") (unit 1) (value "WS2812D") (footprint "LED_SMD:LED_WS2812D-F5-1261_5.8x8.6mm_P1.1mm")
     )
     (path "/2340e06d-ed44-4fa8-887e-cf79108a5c5f"
-      (reference "D10") (unit 1) (value "WS2812D") (footprint "footprints:WS2811-THT-LED")
+      (reference "D10") (unit 1) (value "WS2812D") (footprint "LED_SMD:LED_WS2812D-F5-1261_5.8x8.6mm_P1.1mm")
     )
     (path "/7f961cb0-ab19-4d1c-91cc-5cb89d4cc843"
-      (reference "D11") (unit 1) (value "WS2812D") (footprint "footprints:WS2811-THT-LED")
+      (reference "D11") (unit 1) (value "WS2812D") (footprint "LED_SMD:LED_WS2812D-F5-1261_5.8x8.6mm_P1.1mm")
     )
     (path "/5b2787cf-10ba-40ef-8f60-4e71bb9c23ea"
-      (reference "D12") (unit 1) (value "WS2812D") (footprint "footprints:WS2811-THT-LED")
+      (reference "D12") (unit 1) (value "WS2812D") (footprint "LED_SMD:LED_WS2812D-F5-1261_5.8x8.6mm_P1.1mm")
     )
     (path "/d71593f7-09cf-4465-9cce-fd2751f1f4fa"

Commit message: new 3d for encoder, fixing ibom.html + new images
Parts:
- C1, C10, C4, C7: value 33n -> 100n
- R1, R10, R11, R12, R2, R21, R22, R3, R31, R32, R4, R41, R42, R5, R6, R7, R8, R9: Purchase https://www.aliexpress.com/item/1005003021579348.html -> https://www.aliexpress.com/item/32865947306.html

Commit message: adding v0.7
Parts:
- C1, C10, C21, C31, C4, C41, C7: Purchase https://www.aliexpress.com/item/32964553793.html -> (none)
- D1, D10, D11, D12, D2, D3, D4, D5, D6, D7, D8, D9: footprint LED_SMD:LED_WS2812D-F5-1261_5.8x8.6mm_P1.1mm -> andilge KiCad footprints:WS2811D-F5-1261; Purchase https://www.aliexpress.com/item/32790928817.html -> (none)
- J1: Purchase https://www.aliexpress.com/item/32853351049.html -> (none)
- R1, R10, R11, R12, R2, R21, R22, R3, R31, R32, R4, R41, R42, R5, R6, R7, R8, R9: Purchase https://www.aliexpress.com/item/32865947306.html -> (none)
- R33, R43: Purchase https://www.aliexpress.com/item/1005003021579348.html -> (none)

Commit message: adding fabrication files for 0.7
Parts:
- C1, C10, C21, C31, C4, C41, C7: Purchase (none) -> https://www.aliexpress.com/item/32964553793.html
- D1, D10, D11, D12, D2, D3, D4, D5, D6, D7, D8, D9: value WS2812D -> WS2812D F5 hat; Purchase (none) -> https://www.aliexpress.com/item/32790928817.html
- J1: Purchase (none) -> https://www.aliexpress.com/item/32853351049.html
- R1, R10, R11, R12, R2, R21, R22, R3, R31, R32, R33, R4, R41, R42, R43, R5, R6, R7, R8, R9: Purchase (none) -> https://www.aliexpress.com/item/1005003021579348.html
