File: Futai Encoder + WS2811 ring.kicad_sch (KiCad schematic)
At the start: 41 parts, among them J1 Conn_02x05_Top_Bottom, SW1 RotaryEncoder_Switch_RGB

Commit message: lowering value for R1-R12
Parts:
- R1, R10, R11, R12, R2, R3, R4, R5, R6, R7, R8, R9: value 130 -> 68
Changed lines of the file:
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@@
     (in_bom yes) (on_board yes) (fields_autoplaced)
     (property "Reference" "R8" (id 0) (at 102.87 95.25 90))
-    (property "Value" "130" (id 1) (at 102.87 97.79 90))
+    (property "Value" "68" (id 1) (at 102.87 97.79 90))
     (property "Footprint" "Resistor_SMD:R_0805_2012Metric" (id 2) (at 102.87 101.6 0)
       (effects (font (size 1.27 1.27)) hide)
@@
     (in_bom yes) (on_board yes) (fields_autoplaced)
     (property "Reference" "R10" (id 0) (at 120.65 125.73 90))
-    (property "Value" "130" (id 1) (at 120.65 128.27 90))
+    (property "Value" "68" (id 1) (at 120.65 128.27 90))
     (property "Footprint" "Resistor_SMD:R_0805_2012Metric" (id 2) (at 120.65 132.08 0)
       (effects (font (size 1.27 1.27)) hide)
@@
     (in_bom yes) (on_board yes) (fields_autoplaced)
     (property "Reference" "R3" (id 0) (at 120.65 34.29 90))
-    (property "Value" "130" (id 1) (at 120.65 36.83 90))
+    (property "Value" "68" (id 1) (at 120.65 36.83 90))
     (property "Footprint" "Resistor_SMD:R_0805_2012Metric" (id 2) (at 120.65 40.64 0)
       (effects (font (size 1.27 1.27)) hide)
@@
     (in_bom yes) (on_board yes) (fields_autoplaced)
     (property "Reference" "R5" (id 0) (at 102.87 64.77 90))
-    (property "Value" "130" (id 1) (at 102.87 67.31 90))
+    (property "Value" "68" (id 1) (at 102.87 67.31 90))
     (property "Footprint" "Resistor_SMD:R_0805_2012Metric" (id 2) (at 102.87 71.12 0)
       (effects (font (size 1.27 1.27)) hide)
@@
     (in_bom yes) (on_board yes) (fields_autoplaced)
     (property "Reference" "R6" (id 0) (at 85.09 64.77 90))
-    (property "Value" "130" (id 1) (at 85.09 67.31 90))
+    (property "Value" "68" (id 1) (at 85.09 67.31 90))
     (property "Footprint" "Resistor_SMD:R_0805_2012Metric" (id 2) (at 85.09 71.12 0)
       (effects (font (size 1.27 1.27)) hide)
@@
     (in_bom yes) (on_board yes) (fields_autoplaced)
     (property "Reference" "R9" (id 0) (at 120.65 95.25 90))
-    (property "Value" "130" (id 1) (at 120.65 97.79 90))
+    (property "Value" "68" (id 1) (at 120.65 97.79 90))
     (property "Footprint" "Resistor_SMD:R_0805_2012Metric" (id 2) (at 120.65 101.6 0)
       (effects (font (size 1.27 1.27)) hide)
@@
     (in_bom yes) (on_board yes) (fields_autoplaced)
     (property "Reference" "R1" (id 0) (at 85.09 34.29 90))
-    (property "Value" "130" (id 1) (at 85.09 36.83 90))
+    (property "Value" "68" (id 1) (at 85.09 36.83 90))
     (property "Footprint" "Resistor_SMD:R_0805_2012Metric" (id 2) (at 85.09 40.64 0)
       (effects (font (size 1.27 1.27)) hide)
@@
     (in_bom yes) (on_board yes) (fields_autoplaced)
     (property "Reference" "R4" (id 0) (at 120.65 64.77 90))
-    (property "Value" "130" (id 1) (at 120.65 67.31 90))
+    (property "Value" "68" (id 1) (at 120.65 67.31 90))
     (property "Footprint" "Resistor_SMD:R_0805_2012Metric" (id 2) (at 120.65 71.12 0)
       (effects (font (size 1.27 1.27)) hide)
@@
     (in_bom yes) (on_board yes) (fields_autoplaced)
     (property "Reference" "R12" (id 0) (at 85.09 125.73 90))
-    (property "Value" "130" (id 1) (at 85.09 128.27 90))
+    (property "Value" "68" (id 1) (at 85.09 128.27 90))
     (property "Footprint" "Resistor_SMD:R_0805_2012Metric" (id 2) (at 85.09 132.08 0)
       (effects (font (size 1.27 1.27)) hide)
@@
     (in_bom yes) (on_board yes) (fields_autoplaced)
     (property "Reference" "R2" (id 0) (at 102.87 34.29 90))
-    (property "Value" "130" (id 1) (at 102.87 36.83 90))
+    (property "Value" "68" (id 1) (at 102.87 36.83 90))
     (property "Footprint" "Resistor_SMD:R_0805_2012Metric" (id 2) (at 102.87 40.64 0)
       (effects (font (size 1.27 1.27)) hide)
@@
     (in_bom yes) (on_board yes) (fields_autoplaced)
     (property "Reference" "R11" (id 0) (at 102.87 125.73 90))
-    (property "Value" "130" (id 1) (at 102.87 128.27 90))
+    (property "Value" "68" (id 1) (at 102.87 128.27 90))
     (property "Footprint" "Resistor_SMD:R_0805_2012Metric" (id 2) (at 102.87 132.08 0)
       (effects (font (size 1.27 1.27)) hide)
@@
     (in_bom yes) (on_board yes) (fields_autoplaced)
     (property "Reference" "R7" (id 0) (at 85.09 95.25 90))
-    (property "Value" "130" (id 1) (at 85.09 97.79 90))
+    (property "Value" "68" (id 1) (at 85.09 97.79 90))
     (property "Footprint" "Resistor_SMD:R_0805_2012Metric" (id 2) (at 85.09 101.6 0)
       (effects (font (size 1.27 1.27)) hide)
@@
     )
     (path "/a1907388-9e00-468a-988b-8992902b3682"
-      (reference "R1") (unit 1) (value "130") (footprint "Resistor_SMD:R_0805_2012Metric")
+      (reference "R1") (unit 1) (value "68") (footprint "Resistor_SMD:R_0805_2012Metric")
     )
     (path "/bd29be46-488e-4e08-b4da-96638cf12682"
-      (reference "R2") (unit 1) (value "130") (footprint "Resistor_SMD:R_0805_2012Metric")
+      (reference "R2") (unit 1) (value "68") (footprint "Resistor_SMD:R_0805_2012Metric")
     )
     (path "/14453a58-5327-4949-b6fd-b66f4b436bab"
-      (reference "R3") (unit 1) (value "130") (footprint "Resistor_SMD:R_0805_2012Metric")
+      (reference "R3") (unit 1) (value "68") (footprint "Resistor_SMD:R_0805_2012Metric")
     )
     (path "/aa5c361e-15bc-43d6-86f2-1ed525ecf6c4"
-      (reference "R4") (unit 1) (value "130") (footprint "Resistor_SMD:R_0805_2012Metric")
+      (reference "R4") (unit 1) (value "68") (footprint "Resistor_SMD:R_0805_2012Metric")
     )
     (path "/777fe8f2-679b-4ab3-8661-f8ea51b30eb5"
-      (reference "R5") (unit 1) (value "130") (footprint "Resistor_SMD:R_0805_2012Metric")
+      (reference "R5") (unit 1) (value "68") (footprint "Resistor_SMD:R_0805_2012Metric")
     )
     (path "/7c6bc579-2e40-428e-8e02-8ea37e169713"
-      (reference "R6") (unit 1) (value "130") (footprint "Resistor_SMD:R_0805_2012Metric")
+      (reference "R6") (unit 1) (value "68") (footprint "Resistor_SMD:R_0805_2012Metric")
     )
     (path "/d3ee32eb-50bd-4159-b780-721a0ef3b763"
-      (reference "R7") (unit 1) (value "130") (footprint "Resistor_SMD:R_0805_2012Metric")
+      (reference "R7") (unit 1) (value "68") (footprint "Resistor_SMD:R_0805_2012Metric")
     )
     (path "/0a22ebe2-19e4-4e44-aec5-220a61f1450f"
-      (reference "R8") (unit 1) (value "130") (footprint "Resistor_SMD:R_0805_2012Metric")
+      (reference "R8") (unit 1) (value "68") (footprint "Resistor_SMD:R_0805_2012Metric")
     )
     (path "/7fdf067d-1b60-4cbc-9f7c-e330736a106f"
-      (reference "R9") (unit 1) (value "130") (footprint "Resistor_SMD:R_0805_2012Metric")
+      (reference "R9") (unit 1) (value "68") (footprint "Resistor_SMD:R_0805_2012Metric")
     )
     (path "/0f303b4e-56c5-4092-86d3-ba3d944a7183"
-      (reference "R10") (unit 1) (value "130") (footprint "Resistor_SMD:R_0805_2012Metric")
+      (reference "R10") (unit 1) (value "68") (footprint "Resistor_SMD:R_0805_2012Metric")
     )
     (path "/bdaf077b-081d-4ce2-9917-9e66a4691edd"
-      (reference "R11") (unit 1) (value "130") (footprint "Resistor_SMD:R_0805_2012Metric")
+      (reference "R11") (unit 1) (value "68") (footprint "Resistor_SMD:R_0805_2012Metric")
     )
     (path "/ab739511-7e26-470d-a2f4-e231c5b21cc6"
-      (reference "R12") (unit 1) (value "130") (footprint "Resistor_SMD:R_0805_2012Metric")
+      (reference "R12") (unit 1) (value "68") (footprint "Resistor_SMD:R_0805_2012Metric")
     )
     (path "/fa9aa5e4-b61f-4a04-b576-5b06f9fd3c52"

Commit message: small change to value R1-R12
Parts:
- R1, R10, R11, R12, R2, R3, R4, R5, R6, R7, R8, R9: value 68 -> 62
Changed lines of the file:
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@@
     (in_bom yes) (on_board yes) (fields_autoplaced)
     (property "Reference" "R8" (id 0) (at 102.87 95.25 90))
-    (property "Value" "68" (id 1) (at 102.87 97.79 90))
+    (property "Value" "62" (id 1) (at 102.87 97.79 90))
     (property "Footprint" "Resistor_SMD:R_0805_2012Metric" (id 2) (at 102.87 101.6 0)
       (effects (font (size 1.27 1.27)) hide)
@@
     (in_bom yes) (on_board yes) (fields_autoplaced)
     (property "Reference" "R10" (id 0) (at 120.65 125.73 90))
-    (property "Value" "68" (id 1) (at 120.65 128.27 90))
+    (property "Value" "62" (id 1) (at 120.65 128.27 90))
     (property "Footprint" "Resistor_SMD:R_0805_2012Metric" (id 2) (at 120.65 132.08 0)
       (effects (font (size 1.27 1.27)) hide)
@@
     (in_bom yes) (on_board yes) (fields_autoplaced)
     (property "Reference" "R3" (id 0) (at 120.65 34.29 90))
-    (property "Value" "68" (id 1) (at 120.65 36.83 90))
+    (property "Value" "62" (id 1) (at 120.65 36.83 90))
     (property "Footprint" "Resistor_SMD:R_0805_2012Metric" (id 2) (at 120.65 40.64 0)
       (effects (font (size 1.27 1.27)) hide)
@@
     (in_bom yes) (on_board yes) (fields_autoplaced)
     (property "Reference" "R5" (id 0) (at 102.87 64.77 90))
-    (property "Value" "68" (id 1) (at 102.87 67.31 90))
+    (property "Value" "62" (id 1) (at 102.87 67.31 90))
     (property "Footprint" "Resistor_SMD:R_0805_2012Metric" (id 2) (at 102.87 71.12 0)
       (effects (font (size 1.27 1.27)) hide)
@@
     (in_bom yes) (on_board yes) (fields_autoplaced)
     (property "Reference" "R6" (id 0) (at 85.09 64.77 90))
-    (property "Value" "68" (id 1) (at 85.09 67.31 90))
+    (property "Value" "62" (id 1) (at 85.09 67.31 90))
     (property "Footprint" "Resistor_SMD:R_0805_2012Metric" (id 2) (at 85.09 71.12 0)
       (effects (font (size 1.27 1.27)) hide)
@@
     (in_bom yes) (on_board yes) (fields_autoplaced)
     (property "Reference" "R9" (id 0) (at 120.65 95.25 90))
-    (property "Value" "68" (id 1) (at 120.65 97.79 90))
+    (property "Value" "62" (id 1) (at 120.65 97.79 90))
     (property "Footprint" "Resistor_SMD:R_0805_2012Metric" (id 2) (at 120.65 101.6 0)
       (effects (font (size 1.27 1.27)) hide)
@@
     (in_bom yes) (on_board yes) (fields_autoplaced)
     (property "Reference" "R1" (id 0) (at 85.09 34.29 90))
-    (property "Value" "68" (id 1) (at 85.09 36.83 90))
+    (property "Value" "62" (id 1) (at 85.09 36.83 90))
     (property "Footprint" "Resistor_SMD:R_0805_2012Metric" (id 2) (at 85.09 40.64 0)
       (effects (font (size 1.27 1.27)) hide)
@@
     (in_bom yes) (on_board yes) (fields_autoplaced)
     (property "Reference" "R4" (id 0) (at 120.65 64.77 90))
-    (property "Value" "68" (id 1) (at 120.65 67.31 90))
+    (property "Value" "62" (id 1) (at 120.65 67.31 90))
     (property "Footprint" "Resistor_SMD:R_0805_2012Metric" (id 2) (at 120.65 71.12 0)
       (effects (font (size 1.27 1.27)) hide)
@@
     (in_bom yes) (on_board yes) (fields_autoplaced)
     (property "Reference" "R12" (id 0) (at 85.09 125.73 90))
-    (property "Value" "68" (id 1) (at 85.09 128.27 90))
+    (property "Value" "62" (id 1) (at 85.09 128.27 90))
     (property "Footprint" "Resistor_SMD:R_0805_2012Metric" (id 2) (at 85.09 132.08 0)
       (effects (font (size 1.27 1.27)) hide)
@@
     (in_bom yes) (on_board yes) (fields_autoplaced)
     (property "Reference" "R2" (id 0) (at 102.87 34.29 90))
-    (property "Value" "68" (id 1) (at 102.87 36.83 90))
+    (property "Value" "62" (id 1) (at 102.87 36.83 90))
     (property "Footprint" "Resistor_SMD:R_0805_2012Metric" (id 2) (at 102.87 40.64 0)
       (effects (font (size 1.27 1.27)) hide)
@@
     (in_bom yes) (on_board yes) (fields_autoplaced)
     (property "Reference" "R11" (id 0) (at 102.87 125.73 90))
-    (property "Value" "68" (id 1) (at 102.87 128.27 90))
+    (property "Value" "62" (id 1) (at 102.87 128.27 90))
     (property "Footprint" "Resistor_SMD:R_0805_2012Metric" (id 2) (at 102.87 132.08 0)
       (effects (font (size 1.27 1.27)) hide)
@@
     (in_bom yes) (on_board yes) (fields_autoplaced)
     (property "Reference" "R7" (id 0) (at 85.09 95.25 90))
-    (property "Value" "68" (id 1) (at 85.09 97.79 90))
+    (property "Value" "62" (id 1) (at 85.09 97.79 90))
     (property "Footprint" "Resistor_SMD:R_0805_2012Metric" (id 2) (at 85.09 101.6 0)
       (effects (font (size 1.27 1.27)) hide)
@@
     )
     (path "/a1907388-9e00-468a-988b-8992902b3682"
-      (reference "R1") (unit 1) (value "68") (footprint "Resistor_SMD:R_0805_2012Metric")
+      (reference "R1") (unit 1) (value "62") (footprint "Resistor_SMD:R_0805_2012Metric")
     )
     (path "/bd29be46-488e-4e08-b4da-96638cf12682"
-      (reference "R2") (unit 1) (value "68") (footprint "Resistor_SMD:R_0805_2012Metric")
+      (reference "R2") (unit 1) (value "62") (footprint "Resistor_SMD:R_0805_2012Metric")
     )
     (path "/14453a58-5327-4949-b6fd-b66f4b436bab"
-      (reference "R3") (unit 1) (value "68") (footprint "Resistor_SMD:R_0805_2012Metric")
+      (reference "R3") (unit 1) (value "62") (footprint "Resistor_SMD:R_0805_2012Metric")
     )
     (path "/aa5c361e-15bc-43d6-86f2-1ed525ecf6c4"
-      (reference "R4") (unit 1) (value "68") (footprint "Resistor_SMD:R_0805_2012Metric")
+      (reference "R4") (unit 1) (value "62") (footprint "Resistor_SMD:R_0805_2012Metric")
     )
     (path "/777fe8f2-679b-4ab3-8661-f8ea51b30eb5"
-      (reference "R5") (unit 1) (value "68") (footprint "Resistor_SMD:R_0805_2012Metric")
+      (reference "R5") (unit 1) (value "62") (footprint "Resistor_SMD:R_0805_2012Metric")
     )
     (path "/7c6bc579-2e40-428e-8e02-8ea37e169713"
-      (reference "R6") (unit 1) (value "68") (footprint "Resistor_SMD:R_0805_2012Metric")
+      (reference "R6") (unit 1) (value "62") (footprint "Resistor_SMD:R_0805_2012Metric")
     )
     (path "/d3ee32eb-50bd-4159-b780-721a0ef3b763"
-      (reference "R7") (unit 1) (value "68") (footprint "Resistor_SMD:R_0805_2012Metric")
+      (reference "R7") (unit 1) (value "62") (footprint "Resistor_SMD:R_0805_2012Metric")
     )
     (path "/0a22ebe2-19e4-4e44-aec5-220a61f1450f"
-      (reference "R8") (unit 1) (value "68") (footprint "Resistor_SMD:R_0805_2012Metric")
+      (reference "R8") (unit 1) (value "62") (footprint "Resistor_SMD:R_0805_2012Metric")
     )
     (path "/7fdf067d-1b60-4cbc-9f7c-e330736a106f"
-      (reference "R9") (unit 1) (value "68") (footprint "Resistor_SMD:R_0805_2012Metric")
+      (reference "R9") (unit 1) (value "62") (footprint "Resistor_SMD:R_0805_2012Metric")
     )
     (path "/0f303b4e-56c5-4092-86d3-ba3d944a7183"
-      (reference "R10") (unit 1) (value "68") (footprint "Resistor_SMD:R_0805_2012Metric")
+      (reference "R10") (unit 1) (value "62") (footprint "Resistor_SMD:R_0805_2012Metric")
     )
     (path "/bdaf077b-081d-4ce2-9917-9e66a4691edd"
-      (reference "R11") (unit 1) (value "68") (footprint "Resistor_SMD:R_0805_2012Metric")
+      (reference "R11") (unit 1) (value "62") (footprint "Resistor_SMD:R_0805_2012Metric")
     )
     (path "/ab739511-7e26-470d-a2f4-e231c5b21cc6"
-      (reference "R12") (unit 1) (value "68") (footprint "Resistor_SMD:R_0805_2012Metric")
+      (reference "R12") (unit 1) (value "62") (footprint "Resistor_SMD:R_0805_2012Metric")
     )
     (path "/fa9aa5e4-b61f-4a04-b576-5b06f9fd3c52"

Commit message: v0.8
Parts:
- removed C10, C4: 100n, Capacitor_SMD:C_0805_2012Metric, symbol Device:C_Small
- removed R12: 62, Resistor_SMD:R_0805_2012Metric, symbol Device:R_Small
- added C11, C3, C5, C9: 220n, Capacitor_SMD:C_0805_2012Metric, symbol Device:C_Small
- C1, C7: value 100n -> 220n
- R1, R10, R11, R2, R3, R4, R5, R6, R7, R8, R9: value 62 -> 75
Connections:
- net GND: now also C11.1, C3.2, C5.1, C9.2
- net at D9.1 (DOUT): now also R9.2; no longer D10.4 (DIN)
- net +5VL: now reaches D9.2 (VDD)
- net +5VL: now also C1.1, C7.1, D1.2 (VDD), D10.2 (VDD), D11.2 (VDD), D12.2 (VDD), D2.2 (VDD), D3.2 (VDD), D4.2 (VDD), D5.2 (VDD), D6.2 (VDD), D7.2 (VDD), D8.2 (VDD), J1.5 (Pin_5), R31.1, R41.1, SW1.1 (C+), C11.2, C3.1, C5.2, C9.1; no longer R9.2
- net at D9.4 (DIN): now also R8.1; no longer D8.1 (DOUT)
- net at R8.2: now also D8.1 (DOUT); no longer D8.2 (VDD)
- net at R10.2: now also D11.4 (DIN); no longer D10.2 (VDD)
- net at R3.2: now also D3.1 (DOUT); no longer D3.2 (VDD)
- net at D10.1 (DOUT): now also R10.1; no longer D11.4 (DIN)
- net at D1.1 (DOUT): now also R1.2; no longer D2.4 (DIN)
- net at D7.1 (DOUT): now also R7.2; no longer D8.4 (DIN)
- net at D7.4 (DIN): now also R6.2; no longer D6.1 (DOUT)
- net at R4.2: now also D5.4 (DIN); no longer D4.2 (VDD)
- net at D3.4 (DIN): now also R2.1; no longer D2.1 (DOUT)
- net at R2.2: now also D2.1 (DOUT); no longer D2.2 (VDD)
- net at D12.4 (DIN): now also R11.2; no longer D11.1 (DOUT)
- net at D5.1 (DOUT): now also R5.1; no longer D6.4 (DIN)
- net at R5.2: now also D6.4 (DIN); no longer D5.2 (VDD)
- net at D4.1 (DOUT): now also R4.1; no longer D5.4 (DIN)
- net at D4.4 (DIN): now also R3.1; no longer D3.1 (DOUT)
- removed net +5V: J1.5 (Pin_5), R1.1, R10.1, R11.1, R2.1, R3.1, R31.1, R4.1, R41.1, R5.1, R6.1, R7.1, R8.1, R9.1, SW1.1 (C+)
- new net: D10.4 (DIN), R9.1
- new net: D2.4 (DIN), R1.1
- new net: D11.1 (DOUT), R11.1
- new net: D8.4 (DIN), R7.1
- new net: D6.1 (DOUT), R6.1
Other:
- moved on the sheet: C1, C21, C31, C41, C7, D1, D10, D11, D12, D2, D3, D4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
